Commit message: robot moves!

File: lab_4/ex03/robot_start/src/description/robot.urdf.xacro (robot description, xacro)
@@ -29,13 +29,7 @@
       <material name="blue"/>
     </visual>
-    <collision>
-      <origin xyz="0 0 ${base_z_offset}" rpy="1.5708 0 0"/>
-      <geometry>
-        <cylinder length="${base_length}" radius="${base_radius}"/>
-      </geometry>
-    </collision>
     <inertial>
       <mass value="${base_mass}"/>
-      <inertia ixx="10.0" ixy="0.0" ixz="0.0" iyy="10.0" iyz="0.0" izz="10.0"/>
+      <inertia ixx="0.0024" ixy="0.0" ixz="0.0" iyy="0.0017" iyz="0.0" izz="0.0024"/>
     </inertial>
   </link>
@@ -43,4 +37,5 @@
     <link name="${prefix}_wheel">
       <visual>
+        <origin xyz="0.0 0.0 0.0" rpy="0 0 ${turn_angle}"/>
         <geometry>
           <mesh filename="package://robot_start/meshes/wheel.stl"/>
@@ -56,5 +51,5 @@
       <inertial>
         <mass value="${wheel_mass}"/>
-        <inertia ixx="0.1" ixy="0.0" ixz="0.0" iyy="0.1" iyz="0.0" izz="0.1"/>
+        <inertia ixx="0.000001" ixy="0.0" ixz="0.0" iyy="0.000001" iyz="0.0" izz="0.000002"/>
       </inertial>
     </link>
@@ -62,5 +57,5 @@
       <parent link="base_link"/>
       <child link="${prefix}_wheel"/>
-      <origin xyz="-0.02 ${reflect * 0.06} ${base_z_offset}" rpy="${turn_angle} 0 0"/>
+      <origin xyz="-0.02 ${reflect * 0.06} ${base_z_offset}" rpy="0 0 0"/>
       <axis xyz="0 ${reflect} 0"/>
       <dynamics damping="0.1" friction="0.0"/>
@@ -84,5 +79,5 @@
     <inertial>
       <mass value="${caster_mass}"/>
-      <inertia ixx="0.01" ixy="0.0" ixz="0.0" iyy="0.01" iyz="0.0" izz="0.01"/>
+      <inertia ixx="0.0000016" ixy="0.0" ixz="0.0" iyy="0.0000016" iyz="0.0" izz="0.0000016"/>
     </inertial>
   </link>
