Commit message: robot drives properly

File: lab_4/ex03/robot_start/src/description/robot.gazebo.xacro (robot description, xacro)
@@ -4,6 +4,6 @@
   <gazebo>
     <plugin filename="libgz-sim8-diff-drive-system.so" name="gz::sim::v8::systems::DiffDrive">
-      <left_joint>left_wheel_joint</left_joint>
-      <right_joint>right_wheel_joint</right_joint>
+      <left_joint>right_wheel_joint</left_joint>
+      <right_joint>left_wheel_joint</right_joint>
       <wheel_separation>0.12</wheel_separation>
       <wheel_radius>0.02</wheel_radius>

File: lab_4/ex03/robot_start/src/description/robot.urdf.xacro (robot description, xacro)
@@ -58,10 +58,10 @@
       <child link="${prefix}_wheel"/>
       <origin xyz="-0.02 ${reflect * 0.06} ${base_z_offset}" rpy="0 0 0"/>
-      <axis xyz="0 ${reflect} 0"/>
+      <axis xyz="0 1 0"/>
       <dynamics damping="0.1" friction="0.0"/>
     </joint>
   </xacro:macro>
-  <xacro:wheel prefix="left" reflect="1" turn_angle="0"/>
-  <xacro:wheel prefix="right" reflect="-1" turn_angle="3.1415"/>
+  <xacro:wheel prefix="left" reflect="-1" turn_angle="0"/>
+  <xacro:wheel prefix="right" reflect="1" turn_angle="3.1415"/>
   <link name="front_caster">
     <visual>
